Commit message: creating urdf; bug -- colors not working and coordinates are really messed up

File: cara_description/urdf/cara.urdf (robot description, URDF)
Before this commit: robot cara, 39 links, 38 joints
Links:
- removed link c_clamp_1
- removed link c_clamp_2
- removed link c_clamp_3
- removed link c_clamp_4
- removed link circuit_plate
- removed link feedback
- removed link imu
- removed link lidar_base
- removed link lidar_bottom
- removed link lidar_up
- removed link motor_1
- removed link motor_2
- removed link motor_3
- removed link motor_4
- removed link rplidar_frame
- removed link s1
- removed link s10
- removed link s11
- removed link s12
- removed link s2
- removed link s3
- removed link s4
- removed link s5
- removed link s6
- removed link s7
- removed link s8
- removed link s9
- removed link shaft_1
- removed link shaft_2
- removed link shaft_3
- removed link shaft_4
- removed link top_plate
- removed link wheel_1
- removed link wheel_2
- removed link wheel_3
- removed link wheel_4
- removed link x
- removed link y
- link base_link: mass 8 -> None; geometry visual box size=0.16 0.16 0.12
Joints:
- removed joint base_c_clamp_1
- removed joint base_c_clamp_2
- removed joint base_c_clamp_3
- removed joint base_c_clamp_4
- removed joint base_link_circuit_plate
- removed joint base_link_feedback
- removed joint base_link_imu
- removed joint base_link_rplidar_frame
- removed joint base_link_top_plate
- removed joint base_link_x
- removed joint base_link_y
- removed joint c_clamp_motor_1
- removed joint c_clamp_motor_2
- removed joint c_clamp_motor_3
- removed joint c_clamp_motor_4
- removed joint circuit_plate_lidar_base
- removed joint feedback_s1
- removed joint feedback_s2
- removed joint feedback_s3
- removed joint feedback_s4
- removed joint feedback_s5
- removed joint feedback_s6
- removed joint feedback_s7
- removed joint feedback_s8
- removed joint lidar_base_lidar_bottom
- removed joint lidar_base_s10
- removed joint lidar_base_s11
- removed joint lidar_base_s12
- removed joint lidar_base_s9
- removed joint lidar_bottom_lidar_up
- removed joint motor_shaft_1
- removed joint motor_shaft_2
- removed joint motor_shaft_3
- removed joint motor_shaft_4
- removed joint shaft_wheel_1
- removed joint shaft_wheel_2
- removed joint shaft_wheel_3
- removed joint shaft_wheel_4

Commit message: added in gazebo and joints

File: cara_description/urdf/cara.urdf (robot description, URDF)
Before this commit: robot test_robot, 1 links, 0 joints
Links:
- added link frame; visual mesh filename=package://cara_description/meshes/frame.stl scale=0.001 0.001 0.001
- added link imu; visual box size=0.05 0.03 0.004
- added link imu_frame; visual sphere radius=0.001
- added link lidar_base; visual mesh filename=package://cara_description/meshes/lidar_base.stl scale=0.001 0.001 0.001
- added link lidar_bottom; visual mesh filename=package://cara_description/meshes/lidar_bottom.stl scale=0.001 0.001 0.001
- added link lidar_up; visual mesh filename=package://cara_description/meshes/lidar_up.stl scale=0.001 0.001 0.001
- added link motorL, mass 1; visual mesh filename=package://cara_description/meshes/motor-and-mount.stl scale=.025 .025 .025
- added link motorR, mass 1; visual mesh filename=package://cara_description/meshes/motor-and-mount.stl scale=.025 .025 .025
- added link rplidar_frame; visual sphere radius=0.001
- added link s10; visual mesh filename=package://cara_description/meshes/stud.stl scale=0.001 0.001 0.001
- added link s11; visual mesh filename=package://cara_description/meshes/stud.stl scale=0.001 0.001 0.001
- added link s12; visual mesh filename=package://cara_description/meshes/stud.stl scale=0.001 0.001 0.001
- added link s9; visual mesh filename=package://cara_description/meshes/stud.stl scale=0.001 0.001 0.001
- added link wheelL; visual mesh filename=package://cara_description/meshes/wheel.stl scale=.001 .001 .001
- added link wheelR; visual mesh filename=package://cara_description/meshes/wheel.stl scale=.001 .001 .001
- added link x; visual sphere radius=0.1
- added link y; visual sphere radius=0.1
- link base_link: geometry collision box size=0.6 0.6 0.4048; collision cylinder length=0.205 radius=.07
Joints:
- added joint base_and_motorL: type fixed, parent base_link, child motorL
- added joint base_and_motorR: type fixed, parent base_link, child motorR
- added joint base_link_frame: type fixed, parent base_link, child frame
- added joint base_link_imu: type fixed, parent base_link, child imu
- added joint base_link_imu_frame: type fixed, parent base_link, child imu_frame, origin xyz=0.0 0 0.24 rpy=0 0 0
- added joint base_link_rplidar_frame: type fixed, parent base_link, child rplidar_frame, origin xyz=-0.1246 0 0.28 rpy=0 0 0
- added joint base_link_x: type fixed, parent base_link, child x
- added joint base_link_y: type fixed, parent base_link, child y
- added joint frame_lidar_base: type fixed, parent frame, child lidar_base
- added joint lidar_base_lidar_bottom: type fixed, parent lidar_base, child lidar_bottom
- added joint lidar_base_s10: type fixed, parent lidar_base, child s10
- added joint lidar_base_s11: type fixed, parent lidar_base, child s11
- added joint lidar_base_s12: type fixed, parent lidar_base, child s12
- added joint lidar_base_s9: type fixed, parent lidar_base, child s9
- added joint lidar_bottom_lidar_up: type fixed, parent lidar_bottom, child lidar_up
- added joint motor_and_wheelL: type continuous, parent motorL, child wheelL, axis 0 1 0, limit effort=30 velocity=1.9
- added joint motor_and_wheelR: type continuous, parent motorR, child wheelR, axis 0 1 0, limit effort=30 velocity=1.9

Commit message: final commit

File: cara_description/urdf/cara.urdf (robot description, URDF)
Before this commit: robot cara, 18 links, 17 joints
Joints:
- joint base_link_imu_frame: origin xyz=0.0 0 0.24 rpy=0 0 0 -> xyz=0.0 0 -0.24 rpy=0 0 0
- joint motor_and_wheelL: limit effort=30 velocity=1.9 -> (none)
- joint motor_and_wheelR: limit effort=30 velocity=1.9 -> (none)
